File: Tarea_2_unai/Tarea_2_unai.kicad_pcb (KiCad board)
At the start: 2 copper layers, 44.5 x 31.5 mm, 10 parts, among them IC2 ESP32-C3-MINI-1-N4X, J1 Conn_01x02_Pin, J2 Conn_01x02_Pin, U1 AMS1117-3.3

Commit message: Sensores añadidos y nuevas capas añadidas
Falta por solucionar el enrutamiento de algunos pines de los sensores
Parts:
- added AC1: ADXL345, Samacsys:CC-14-1, F.Cu at (143.5, 87.5)
- added IC1: DS18B20+, Samacsys:DS18B20, F.Cu at (144.5, 93.5)
- added U2: BMP581, Samacsys:BMP581, F.Cu at (144.2, 79.8)
Connections:
- IC2 pad 13: unconnected-(IC2-IO1-Pad13) -> /Microcontrolador/1WIRE_DATA
- IC2 pad 16: unconnected-(IC2-IO10-Pad16) -> /Microcontrolador/SPI_CS
- IC2 pad 18: unconnected-(IC2-IO4-Pad18) -> /Microcontrolador/SPI_SCK
- IC2 pad 21: unconnected-(IC2-IO7-Pad21) -> /Microcontrolador/SPI_MOSI
- IC2 pad 22: unconnected-(IC2-IO8-Pad22) -> /Microcontrolador/I2C_SDA
- IC2 pad 23: unconnected-(IC2-IO9-Pad23) -> /Microcontrolador/I2C_SCL
- IC2 pad 36: unconnected-(IC2-GND_5-Pad36) -> /Alimentacion/GND_REF
- IC2 pad 37: unconnected-(IC2-GND_6-Pad37) -> /Alimentacion/GND_REF
- IC2 pad 38: unconnected-(IC2-GND_7-Pad38) -> /Alimentacion/GND_REF
- IC2 pad 39: unconnected-(IC2-GND_8-Pad39) -> /Alimentacion/GND_REF
- IC2 pad 40: unconnected-(IC2-GND_9-Pad40) -> /Alimentacion/GND_REF
- IC2 pad 41: unconnected-(IC2-GND_10-Pad41) -> /Alimentacion/GND_REF
- IC2 pad 42: unconnected-(IC2-GND_11-Pad42) -> /Alimentacion/GND_REF
- IC2 pad 43: unconnected-(IC2-GND_12-Pad43) -> /Alimentacion/GND_REF
- IC2 pad 44: unconnected-(IC2-GND_13-Pad44) -> /Alimentacion/GND_REF
- IC2 pad 45: unconnected-(IC2-GND_14-Pad45) -> /Alimentacion/GND_REF
- IC2 pad 46: unconnected-(IC2-GND_15-Pad46) -> /Alimentacion/GND_REF
- IC2 pad 47: unconnected-(IC2-GND_16-Pad47) -> /Alimentacion/GND_REF
- IC2 pad 48: unconnected-(IC2-GND_17-Pad48) -> /Alimentacion/GND_REF
- IC2 pad 49: unconnected-(IC2-GND_18-Pad49) -> /Alimentacion/GND_REF
- IC2 pad 5: unconnected-(IC2-IO2-Pad5) -> /Microcontrolador/SPI_MISO
- IC2 pad 50: unconnected-(IC2-GND_19-Pad50) -> /Alimentacion/GND_REF
- IC2 pad 51: unconnected-(IC2-GND_20-Pad51) -> /Alimentacion/GND_REF
- IC2 pad 52: unconnected-(IC2-GND_21-Pad52) -> /Alimentacion/GND_REF
- IC2 pad 53: unconnected-(IC2-GND_22-Pad53) -> /Alimentacion/GND_REF
- IC2 pad 54: unconnected-(IC2-GND_23-Pad54) -> /Alimentacion/GND_REF
- IC2 pad 55: unconnected-(IC2-GND_24-Pad55) -> /Alimentacion/GND_REF
- IC2 pad 56: unconnected-(IC2-GND_25-Pad56) -> /Alimentacion/GND_REF
- IC2 pad 57: unconnected-(IC2-GND_26-Pad57) -> /Alimentacion/GND_REF
- IC2 pad 58: unconnected-(IC2-GND_27-Pad58) -> /Alimentacion/GND_REF
- IC2 pad 59: unconnected-(IC2-GND_28-Pad59) -> /Alimentacion/GND_REF
- IC2 pad 60: unconnected-(IC2-GND_29-Pad60) -> /Alimentacion/GND_REF
- IC2 pad 61: unconnected-(IC2-GND_30-Pad61) -> /Alimentacion/GND_REF
Routing:
- net /Microcontrolador/SPI_MISO: track 0.00 -> 36.9 mm
- net /Microcontrolador/SPI_MOSI: track 0.00 -> 17.4 mm
- net /Microcontrolador/SPI_SCK: track 0.00 -> 16.1 mm
- net /Alimentacion/VOUT_3V3: track 18.0 -> 31.9 mm, vias 0 -> 4
- net /Microcontrolador/I2C_SDA: track 0.00 -> 11.6 mm
- net /Microcontrolador/1WIRE_DATA: track 0.00 -> 11.1 mm
- net /Microcontrolador/I2C_SCL: track 0.00 -> 10.5 mm
- net /Microcontrolador/SPI_CS: track 0.00 -> 7.59 mm
- added copper zone on B.Cu, net /Alimentacion/VOUT_3V3
Other:
- board size 44.5 x 31.5 mm -> 52.5 x 31.5 mm
- copper layers 2 -> 4

Commit message: Parte_1_sesion_4
Routing:
- net /Alimentacion/GND_REF: track 0.29 -> 32.2 mm, vias 0 -> 7
- net /Microcontrolador/SPI_MISO: track 36.9 -> 21.1 mm, vias 0 -> 2
- net /Microcontrolador/SPI_CS: track 7.59 -> 21.1 mm, vias 0 -> 2
- net /Microcontrolador/SPI_SCK: track 16.1 -> 21.0 mm, vias 0 -> 2
- net /Microcontrolador/SPI_MOSI: track 17.4 -> 21.1 mm, vias 0 -> 2
- net /Alimentacion/VOUT_3V3: track 31.9 -> 34.6 mm
- net (no net): track 0.00 -> 1.00 mm, vias 0 -> 1
- added copper zone on In1.Cu, net /Alimentacion/GND_REF
